File: eagle/4x4-programmable-keypad.brd (EAGLE design)
At the start: 58.4 x 58.4 mm, 33 parts

Commit message: Update board and schematic
Parts:
- moved R1 54.9 mm to (50.8, 5.08), turned to 180 degrees
- moved R12 54.9 mm to (5.08, 35.6), turned to 180 degrees
- moved R16 54.9 mm to (5.08, 50.8), turned to 180 degrees
- moved R5 54.9 mm to (50.8, 20.3), turned to 180 degrees
- moved R2 34.1 mm to (35.6, 5.08)
- moved R6 34.1 mm to (35.6, 20.3)
- moved R11 34.1 mm to (20.3, 35.6), turned to 180 degrees
- moved R15 34.1 mm to (20.3, 50.8), turned to 180 degrees
- moved R3 15.2 mm to (20.3, 5.08), turned to 180 degrees
- moved R4 15.2 mm to (5.08, 5.08), turned to 180 degrees
- moved R7 15.2 mm to (20.3, 20.3), turned to 180 degrees
- moved R8 15.2 mm to (5.08, 20.3), turned to 180 degrees
- moved R10 15.2 mm to (35.6, 35.6)
- moved R13 15.2 mm to (50.8, 50.8), turned to 180 degrees
- moved R14 15.2 mm to (35.6, 50.8)
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- renumbered U$10 to U13, U$11 to U15, U$12 to U11, U$13 to U7, U$14 to U3, U$15 to U16, U$16 to U12, U$17 to U8, U$18 to U4, U$3 to U2, U$4 to U6, U$5 to U10, U$6 to U14, U$7 to U1, U$8 to U5, U$9 to U9
Connections:
- removed net N10: R1.1, U15.1, U15.2
- removed net N14: R3.1, U7.1, U7.2
- removed net N15: R4.1, U3.1, U3.2
- removed net N16: R2.1, U11.1, U11.2
- removed net N18: R5.1, U16.1, U16.2
- removed net N19: R6.1, U12.1, U12.2
- removed net N2: R16.2, U2.1, U2.2
- removed net N20: R7.1, U8.1, U8.2
- removed net N21: R8.1, U4.1, U4.2
- removed net N3: R12.2, U1.1, U1.2
- removed net N4: R15.2, U6.1, U6.2
- removed net N5: R11.2, U5.1, U5.2
- removed net N6: R10.2, U9.1, U9.2
- removed net N7: R9.2, U13.1, U13.2
- removed net N8: R14.2, U10.1, U10.2
- removed net N9: R13.2, U14.1, U14.2
- net D10: now also R14.2, U14.1, U14.2; no longer R13.1
- net D14: now also R10.2, U10.1, U10.2; no longer R14.1
- net D15: now also R9.1, U9.1, U9.2; no longer R10.1
- net D16: now also R13.1, U13.1, U13.2; no longer R9.1
- net D18: now also R5.1, U5.1, U5.2; no longer R11.1
- net D19: now also R6.2, U6.1, U6.2; no longer R15.1
- net D2: now also R3.1, U3.1, U3.2; no longer R4.2
- net D20: now also R1.1, U1.1, U1.2; no longer R12.1
- net D21: now also R2.2, U2.1, U2.2; no longer R16.1
- net D3: now also R4.2, U4.1, U4.2; no longer R3.2
- net D4: now also R7.1, U7.1, U7.2; no longer R2.2
- net D5: now also R8.2, U8.1, U8.2; no longer R1.2
- net D6: now also R11.1, U11.1, U11.2; no longer R8.2
- net D7: now also R12.2, U12.1, U12.2; no longer R7.2
- net D8: now also R15.1, U15.1, U15.2; no longer R6.2
- net D9: now also R16.2, U16.1, U16.2; no longer R5.2
- net GND: now also R1.2, R10.1, R11.2, R12.1, R13.2, R14.1, R15.2, R16.1, R2.1, R3.2, R4.1, R5.2, R6.1, R7.2, R8.1, R9.2; no longer U1.3, U1.4, U10.3, U10.4, U11.3, U11.4, U12.3, U12.4, U13.3, U13.4, U14.3, U14.4, U15.3, U15.4, U16.3, U16.4, U2.3, U2.4, U3.3, U3.4, U4.3, U4.4, U5.3, U5.4, U6.3, U6.4, U7.3, U7.4, U8.3, U8.4, U9.3, U9.4
- net VCC: now also U1.3, U1.4, U10.3, U10.4, U11.3, U11.4, U12.3, U12.4, U13.3, U13.4, U14.3, U14.4, U15.3, U15.4, U16.3, U16.4, U2.3, U2.4, U3.3, U3.4, U4.3, U4.4, U5.3, U5.4, U6.3, U6.4, U7.3, U7.4, U8.3, U8.4, U9.3, U9.4
Routing:
- net VCC: track 0.00 -> 273.2 mm
- net GND: track 0.00 -> 30.5 mm, vias 0 -> 2
- net D5: track 33.0 -> 16.6 mm
- net D8: track 13.6 -> 29.2 mm
- net D3: track 8.35 -> 19.1 mm
- net N14: track 7.79 -> 0.00 mm
- net N9: track 7.67 -> 0.00 mm
- net N8: track 7.67 -> 0.00 mm
- net N6: track 7.67 -> 0.00 mm
- net N7: track 7.67 -> 0.00 mm
- net N5: track 7.67 -> 0.00 mm
- net N4: track 7.67 -> 0.00 mm
- net N3: track 7.67 -> 0.00 mm
- net N2: track 7.67 -> 0.00 mm
- net N20: track 7.67 -> 0.00 mm
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