File: eagle/4x4-programmable-keypad.sch (EAGLE design)
At the start: 33 parts

Commit message: Update board and schematic
Parts:
- removed U$10, U$11, U$12, U$13, U$14, U$15, U$16, U$17, U$18, U$3, U$4, U$5, U$6, U$7, U$8, U$9: TACTILE_BUTTON_6X6X9.5, Pat Sonstiges:TACTILE_BUTTON_6X6X9.5
- added U1, U10, U11, U12, U13, U14, U15, U16, U2, U3, U4, U5, U6, U7, U8, U9: TACTILE_BUTTON_6X6X9.5, Pat Sonstiges:TACTILE_BUTTON_6X6X9.5
Connections:
- removed net N10: R1.1, U$11.1, U$11.3
- removed net N14: R3.1, U$13.1, U$13.3
- removed net N15: R4.1, U$14.1, U$14.3
- removed net N16: R2.1, U$12.1, U$12.3
- removed net N18: R5.1, U$15.1, U$15.3
- removed net N19: R6.1, U$16.1, U$16.3
- removed net N2: R16.2, U$3.1, U$3.3
- removed net N20: R7.1, U$17.1, U$17.3
- removed net N21: R8.1, U$18.1, U$18.3
- removed net N3: R12.2, U$7.1, U$7.3
- removed net N4: R15.2, U$4.1, U$4.3
- removed net N5: R11.2, U$8.1, U$8.3
- removed net N6: R10.2, U$9.1, U$9.3
- removed net N7: R9.2, U$10.1, U$10.3
- removed net N8: R14.2, U$5.1, U$5.3
- removed net N9: R13.2, U$6.1, U$6.3
- net D10: now also R14.2, U14.1, U14.3; no longer R13.1
- net D14: now also R10.2, U10.1, U10.3; no longer R14.1
- net D15: now also R9.1, U9.1, U9.3; no longer R10.1
- net D16: now also R13.1, U13.1, U13.3; no longer R9.1
- net D18: now also R5.1, U5.1, U5.3; no longer R11.1
- net D19: now also R6.2, U6.1, U6.3; no longer R15.1
- net D2: now also R3.1, U3.1, U3.3; no longer R4.2
- net D20: now also R1.1, U1.1, U1.3; no longer R12.1
- net D21: now also R2.2, U2.1, U2.3; no longer R16.1
- net D3: now also R4.2, U4.1, U4.3; no longer R3.2
- net D4: now also R7.1, U7.1, U7.3; no longer R2.2
- net D5: now also R8.2, U8.1, U8.3; no longer R1.2
- net D6: now also R11.1, U11.1, U11.3; no longer R8.2
- net D7: now also R12.2, U12.1, U12.3; no longer R7.2
- net D8: now also R15.1, U15.1, U15.3; no longer R6.2
- net D9: now also R16.2, U16.1, U16.3; no longer R5.2
- net GND: now also R1.2, R10.1, R11.2, R12.1, R13.2, R14.1, R15.2, R16.1, R2.1, R3.2, R4.1, R5.2, R6.1, R7.2, R8.1, R9.2; no longer U$10.2, U$10.4, U$11.2, U$11.4, U$12.2, U$12.4, U$13.2, U$13.4, U$14.2, U$14.4, U$15.2, U$15.4, U$16.2, U$16.4, U$17.2, U$17.4, U$18.2, U$18.4, U$3.2, U$3.4, U$4.2, U$4.4, U$5.2, U$5.4, U$6.2, U$6.4, U$7.2, U$7.4, U$8.2, U$8.4, U$9.2, U$9.4
- net VCC: now also U1.2, U1.4, U10.2, U10.4, U11.2, U11.4, U12.2, U12.4, U13.2, U13.4, U14.2, U14.4, U15.2, U15.4, U16.2, U16.4, U2.2, U2.4, U3.2, U3.4, U4.2, U4.4, U5.2, U5.4, U6.2, U6.4, U7.2, U7.4, U8.2, U8.4, U9.2, U9.4
